File: ArduinoProject/elektronics/arduino_unoModulo/ATMEGA328P.sch (KiCad schematic (older format))
At the start: 9 parts, among them SW1 RESET_SWITCH, U5 ATMEGA328P, X2 CSTCE16MOV53-R0

Commit message: arduino_uno gewijzigd
Parts:
- U5: symbol ATMEGA328P-PU -> ATMEGA328P-PU-RESCUE-Arduino_Uno_R3_From_Scratch
Changed lines of the file:
@@
 EESchema Schematic File Version 2
 LIBS:Arduino_Uno_R3_From_Scratch-rescue
+LIBS:power
+LIBS:device
+LIBS:transistors
+LIBS:conn
+LIBS:linear
+LIBS:regul
+LIBS:74xx
+LIBS:cmos4000
+LIBS:adc-dac
+LIBS:memory
+LIBS:xilinx
+LIBS:microcontrollers
+LIBS:dsp
+LIBS:microchip
+LIBS:analog_switches
+LIBS:motorola
+LIBS:texas
+LIBS:intel
+LIBS:audio
+LIBS:interface
+LIBS:digital-audio
+LIBS:philips
+LIBS:display
+LIBS:cypress
+LIBS:siliconi
+LIBS:opto
+LIBS:atmel
+LIBS:contrib
+LIBS:valves
 LIBS:Arduino_Uno_R3_From_Scratch
 LIBS:MFN_Atmel
@@
 $EndDescr
 $Comp
-L ATMEGA328P-PU U5
+L ATMEGA328P-PU-RESCUE-Arduino_Uno_R3_From_Scratch U5
 U 1 1 55E8A80E
 P 7050 3750
+AR Path="/55E8A80E" Ref="U5"  Part="1"
+AR Path="/55E89CE4/55E8A80E" Ref="U5"  Part="1"
 F 0 "U5" H 6075 1350 60  0000 C CNN
 F 1 "ATMEGA328P" H 7050 6300 60  0000 C CNN
@@
 AREF
 Wire Wire Line
-	4800 3750 5100 3750
-Wire Wire Line
-	5100 3750 5850 3750
-$Comp
-L GND #PWR040
+	4800 3750 5850 3750
+$Comp
+L GND #PWR020
 U 1 1 55E8AA8C
 P 5600 6050
-F 0 "#PWR040" H 5600 6050 30  0001 C CNN
+F 0 "#PWR020" H 5600 6050 30  0001 C CNN
 F 1 "GND" H 5600 5980 30  0001 C CNN
 F 2 "~" H 5600 6050 60  0000 C CNN
@@
 $EndComp
 Wire Wire Line
-	5600 4300 5600 4500
-Wire Wire Line
-	5600 4500 5600 4700
-Wire Wire Line
-	5600 4700 5600 4950
+	5600 4300 5600 4950
 Wire Wire Line
 	5600 4500 5850 4500
@@
 	5850 5500 5600 5500
 Wire Wire Line
-	5600 5250 5600 5500
-Wire Wire Line
-	5600 5500 5600 5700
-Wire Wire Line
-	5600 5700 5600 6050
+	5600 5250 5600 6050
 Wire Wire Line
 	5850 5700 5600 5700
@@
 	5100 4300 5100 4550
 Wire Wire Line
-	8250 6100 8400 6100
-Wire Wire Line
-	8400 6100 9350 6100
-Wire Wire Line
-	8250 5900 8550 5900
-Wire Wire Line
-	8550 5900 9350 5900
+	8250 6100 9350 6100
+Wire Wire Line
+	8250 5900 9350 5900
 Text HLabel 9350 3250 2    40   Input ~ 0
 ARD_AN5/SCL
@@
 	9350 2100 8250 2100
 Wire Wire Line
-	8250 1900 8400 1900
-Wire Wire Line
-	8400 1900 9350 1900
-Wire Wire Line
-	8250 1700 8400 1700
-Wire Wire Line
-	8400 1700 9350 1700
-Wire Wire Line
-	8250 1500 8400 1500
-Wire Wire Line
-	8400 1500 9350 1500
+	8250 1900 9350 1900
+Wire Wire Line
+	8250 1700 9350 1700
+Wire Wire Line
+	8250 1500 9350 1500
 Text HLabel 9350 750  2    40   Input ~ 0
 328P_RESET
 Wire Wire Line
-	3200 1500 3400 1500
-Wire Wire Line
-	3400 1500 4900 1500
-Wire Wire Line
-	4900 1500 5300 1500
-Wire Wire Line
-	5300 1500 5650 1500
-Wire Wire Line
-	5650 1500 5850 1500
+	3200 1500 5850 1500
 $Comp
 L CONN_02X03 ICSP2
@@
 $EndComp
 Wire Wire Line
-	4900 650  4900 750
-Wire Wire Line
-	4900 750  4900 1050
+	4900 650  4900 1050
 Wire Wire Line
 	5300 1350 5300 1500
@@
 Connection ~ 4900 750
 Wire Wire Line
-	4050 750  4900 750
-Wire Wire Line
-	4900 750  5300 750
+	4050 750  5300 750
 Wire Wire Line
 	4350 950  4350 1100
@@
 	3200 950  3200 1500
 $Comp
-L 5V_LDO #PWR041
+L 5V_LDO #PWR021
 U 1 1 55E95BB4
 P 4900 650
-F 0 "#PWR041" H 4900 740 20  0001 C CNN
+F 0 "#PWR021" H 4900 740 20  0001 C CNN
 F 1 "5V_LDO" H 4900 770 30  0000 C CNN
 F 2 "~" H 4900 650 60  0000 C CNN
@@
 $EndComp
 $Comp
-L 5V_LDO #PWR042
+L 5V_LDO #PWR022
 U 1 1 55E95BC3
 P 5600 4300
-F 0 "#PWR042" H 5600 4390 20  0001 C CNN
+F 0 "#PWR022" H 5600 4390 20  0001 C CNN
 F 1 "5V_LDO" H 5600 4420 30  0000 C CNN
 F 2 "~" H 5600 4300 60  0000 C CNN
@@
 $EndComp
 Wire Wire Line
-	5300 2050 5650 2050
-Wire Wire Line
-	5650 2050 5850 2050
+	5300 2050 5850 2050
 Wire Wire Line
 	5300 2050 5300 2150
@@
 	5300 2950 5300 3050
 Wire Wire Line
-	5300 3050 5650 3050
-Wire Wire Line
-	5650 3050 5850 3050
+	5300 3050 5850 3050
 Wire Wire Line
 	5050 2550 4750 2550
@@
 	3500 1650 3500 1775
 Wire Wire Line
-	3300 1650 3400 1650
-Wire Wire Line
-	3400 1650 3500 1650
+	3300 1650 3500 1650
 Wire Wire Line
 	3300 1775 3300 1650
@@
 	3500 2275 3500 2175
 Wire Wire Line
-	3300 2275 3400 2275
-Wire Wire Line
-	3400 2275 3500 2275
+	3300 2275 3500 2275
 Wire Wire Line
 	3300 2275 3300 2175
 $Comp
-L GND #PWR043
+L GND #PWR023
 U 1 1 562077A6
 P 5100 4550
-F 0 "#PWR043" H 5100 4550 30  0001 C CNN
+F 0 "#PWR023" H 5100 4550 30  0001 C CNN
 F 1 "GND" H 5100 4480 30  0001 C CNN
 F 2 "~" H 5100 4550 60  0000 C CNN
@@
 $EndComp
 $Comp
-L GND #PWR044
+L GND #PWR024
 U 1 1 56207870
 P 4750 2900
-F 0 "#PWR044" H 4750 2900 30  0001 C CNN
+F 0 "#PWR024" H 4750 2900 30  0001 C CNN
 F 1 "GND" H 4750 2830 30  0001 C CNN
 F 2 "~" H 4750 2900 60  0000 C CNN
@@
 $EndComp
 $Comp
-L GND #PWR045
+L GND #PWR025
 U 1 1 562079B8
 P 3400 2425
-F 0 "#PWR045" H 3400 2425 30  0001 C CNN
+F 0 "#PWR025" H 3400 2425 30  0001 C CNN
 F 1 "GND" H 3400 2355 30  0001 C CNN
 F 2 "~" H 3400 2425 60  0000 C CNN
@@
 $EndComp
 $Comp
-L GND #PWR047
+L GND #PWR026
 U 1 1 56208C49
 P 4350 1100
-F 0 "#PWR047" H 4350 1100 30  0001 C CNN
+F 0 "#PWR026" H 4350 1100 30  0001 C CNN
 F 1 "GND" H 4350 1030 30  0001 C CNN
 F 2 "~" H 4350 1100 60  0000 C CNN
