File: ArduinoProject/elektronics/arduino_unoModulo/Arduino_Uno_R3_From_Scratch.sch (KiCad schematic (older format))
At the start: 0 parts

Commit message: arduino_uno gewijzigd
Changed lines of the file:
@@
 EESchema Schematic File Version 2
 LIBS:Arduino_Uno_R3_From_Scratch-rescue
+LIBS:power
+LIBS:device
+LIBS:transistors
+LIBS:conn
+LIBS:linear
+LIBS:regul
+LIBS:74xx
+LIBS:cmos4000
+LIBS:adc-dac
+LIBS:memory
+LIBS:xilinx
+LIBS:microcontrollers
+LIBS:dsp
+LIBS:microchip
+LIBS:analog_switches
+LIBS:motorola
+LIBS:texas
+LIBS:intel
+LIBS:audio
+LIBS:interface
+LIBS:digital-audio
+LIBS:philips
+LIBS:display
+LIBS:cypress
+LIBS:siliconi
+LIBS:opto
+LIBS:atmel
+LIBS:contrib
+LIBS:valves
 LIBS:Arduino_Uno_R3_From_Scratch
 LIBS:MFN_Atmel
@@
 F1 "ATMEGA328P.sch" 50
 F2 "AREF" I R 7050 2700 60
-F3 "SERIAL_Rx" I L 5550 3900 60
-F4 "SERIAL_Tx" I L 5550 4150 60
-F5 "ARD_AN5/SCL" I R 7050 5150 60
-F6 "ARD_AN4/SDA" I R 7050 5300 60
-F7 "ARD_AN3" I R 7050 5450 60
-F8 "ARD_AN2" I R 7050 5600 60
-F9 "ARD_AN1" I R 7050 5750 60
-F10 "ARD_AN0" I R 7050 5900 60
-F11 "ARD_DIG7" I R 7050 3850 60
-F12 "ARD_DIG6" I R 7050 4000 60
-F13 "ARD_DIG5" I R 7050 4150 60
-F14 "ARD_DIG4" I R 7050 4300 60
-F15 "ARD_DIG3" I R 7050 4450 60
-F16 "ARD_DIG2" I R 7050 4600 60
-F17 "ARD_DIG1" I R 7050 4750 60
-F18 "ARD_DIG0" I R 7050 4900 60
-F19 "ARD_DIG8" I R 7050 3600 60
-F20 "ARD_DIG9" I R 7050 3450 60
-F21 "ARD_DIG10/SPI_SS" I R 7050 3300 60
-F22 "ARD_DIG11/SPI_MOSI" I R 7050 3150 60
-F23 "ARD_DIG12/SPI_MISO" I R 7050 3000 60
-F24 "ARD_DIG13/SPI_SCK" I R 7050 2850 60
-F25 "328P_RESET" I R 7050 6150 60
+F3 "ARD_AN5/SCL" I R 7050 5150 60
+F4 "ARD_AN4/SDA" I R 7050 5300 60
+F5 "ARD_AN3" I R 7050 5450 60
+F6 "ARD_AN2" I R 7050 5600 60
+F7 "ARD_AN1" I R 7050 5750 60
+F8 "ARD_AN0" I R 7050 5900 60
+F9 "ARD_DIG7" I R 7050 3850 60
+F10 "ARD_DIG6" I R 7050 4000 60
+F11 "ARD_DIG5" I R 7050 4150 60
+F12 "ARD_DIG4" I R 7050 4300 60
+F13 "ARD_DIG3" I R 7050 4450 60
+F14 "ARD_DIG2" I R 7050 4600 60
+F15 "ARD_DIG1" I R 7050 4750 60
+F16 "ARD_DIG0" I R 7050 4900 60
+F17 "ARD_DIG8" I R 7050 3600 60
+F18 "ARD_DIG9" I R 7050 3450 60
+F19 "ARD_DIG10/SPI_SS" I R 7050 3300 60
+F20 "ARD_DIG11/SPI_MOSI" I R 7050 3150 60
+F21 "ARD_DIG12/SPI_MISO" I R 7050 3000 60
+F22 "ARD_DIG13/SPI_SCK" I R 7050 2850 60
+F23 "328P_RESET" I R 7050 6150 60
 $EndSheet
 Wire Wire Line
