File: ArduinoProject/elektronics/arduino_unoModulo/Voltage_Regulator.sch (KiCad schematic (older format))
At the start: 8 parts, among them CON1 BARREL_JACK, U1 LD1117S50TR

Commit message: arduino_uno gewijzigd
Parts:
- D2: symbol LED -> LED-RESCUE-Arduino_Uno_R3_From_Scratch
Changed lines of the file:
@@
 EESchema Schematic File Version 2
 LIBS:Arduino_Uno_R3_From_Scratch-rescue
+LIBS:power
+LIBS:device
+LIBS:transistors
+LIBS:conn
+LIBS:linear
+LIBS:regul
+LIBS:74xx
+LIBS:cmos4000
+LIBS:adc-dac
+LIBS:memory
+LIBS:xilinx
+LIBS:microcontrollers
+LIBS:dsp
+LIBS:microchip
+LIBS:analog_switches
+LIBS:motorola
+LIBS:texas
+LIBS:intel
+LIBS:audio
+LIBS:interface
+LIBS:digital-audio
+LIBS:philips
+LIBS:display
+LIBS:cypress
+LIBS:siliconi
+LIBS:opto
+LIBS:atmel
+LIBS:contrib
+LIBS:valves
 LIBS:Arduino_Uno_R3_From_Scratch
 LIBS:MFN_Atmel
@@
 $EndComp
 $Comp
-L LED D2
+L LED-RESCUE-Arduino_Uno_R3_From_Scratch D2
 U 1 1 55D1FC7B
 P 7800 4125
