File: ArduinoProject/elektronics/sensorModulo/sensorModulo.sch (KiCad schematic (older format))
At the start: 7 parts, among them J1 Conn_01x04_Female, U1 TCRT5000, U2 TCRT5000

Commit message: arduino_uno gewijzigd
Parts:
- R1: renamed from R4; value R -> R56k
- R2: value R -> R56k
- R3: value R -> R220k
- R4: renamed from R1; value R -> R220k
- renumbered U2 to U1, U1 to U2
Changed lines of the file:
@@
 LIBS:valves
 LIBS:tcrt5000
+LIBS:sensorModulo-cache
 EELAYER 25 0
 EELAYER END
@@
 P 3000 4050
 F 0 "R2" V 3080 4050 50  0000 C CNN
-F 1 "R" V 3000 4050 50  0000 C CNN
+F 1 "R56k" V 3000 4050 50  0000 C CNN
 F 2 "" V 2930 4050 50  0001 C CNN
 F 3 "" H 3000 4050 50  0001 C CNN
@@
 $EndComp
 $Comp
-L TCRT5000 U1
+L TCRT5000 U2
 U 1 1 5A047469
 P 3850 4400
-F 0 "U1" H 3850 4400 60  0000 C CNN
+F 0 "U2" H 3850 4400 60  0000 C CNN
 F 1 "TCRT5000" H 3850 4550 60  0000 C CNN
 F 2 "" H 3850 4400 60  0001 C CNN
@@
 $EndComp
 $Comp
-L R R1
+L R R4
 U 1 1 5A047530
 P 4600 4050
-F 0 "R1" V 4680 4050 50  0000 C CNN
-F 1 "R" V 4600 4050 50  0000 C CNN
+F 0 "R4" V 4680 4050 50  0000 C CNN
+F 1 "R220k" V 4600 4050 50  0000 C CNN
 F 2 "" V 4530 4050 50  0001 C CNN
 F 3 "" H 4600 4050 50  0001 C CNN
@@
 	4600 4350 4600 4200
 $Comp
-L R R4
+L R R1
 U 1 1 5A047E13
 P 3000 2450
-F 0 "R4" V 3080 2450 50  0000 C CNN
-F 1 "R" V 3000 2450 50  0000 C CNN
+F 0 "R1" V 3080 2450 50  0000 C CNN
+F 1 "R56k" V 3000 2450 50  0000 C CNN
 F 2 "" V 2930 2450 50  0001 C CNN
 F 3 "" H 3000 2450 50  0001 C CNN
@@
 $EndComp
 $Comp
-L TCRT5000 U2
+L TCRT5000 U1
 U 1 1 5A047E19
 P 3850 2800
-F 0 "U2" H 3850 2800 60  0000 C CNN
+F 0 "U1" H 3850 2800 60  0000 C CNN
 F 1 "TCRT5000" H 3850 2950 60  0000 C CNN
 F 2 "" H 3850 2800 60  0001 C CNN
@@
 P 4600 2450
 F 0 "R3" V 4680 2450 50  0000 C CNN
-F 1 "R" V 4600 2450 50  0000 C CNN
+F 1 "R220k" V 4600 2450 50  0000 C CNN
 F 2 "" V 4530 2450 50  0001 C CNN
 F 3 "" H 4600 2450 50  0001 C CNN
