File: ArduinoProject/elektronics/arduino_unoModulo_tot/Voltage_Regulator.sch (KiCad schematic (older format))
At the start: 8 parts, among them CON1 BARREL_JACK, U1 LD1117S50TR

Commit message: altered kicad
Parts:
- C1: footprint ~ -> ATMEGA328P-AU:QFP80P900X900X120-32N
- C2, C3, CON1, D2, R1: footprint ~ -> (none)
- D1: footprint ~ -> Diodes_SMD:D_0603
- U1: footprint (none) -> LD1117S50TR:SOT230P700X190-4N
Changed lines of the file:
@@
 LIBS:MFN_STMicro
 LIBS:Arduino_Uno_R3_From_Scratch-cache
+LIBS:L298_Driver-cache
 EELAYER 25 0
 EELAYER END
 $Descr A4 11693 8268
 encoding utf-8
-Sheet 2 5
+Sheet 2 6
 Title "Arduino UNO R3 Clone"
 Date "8 oct 2015"
@@
 F 0 "D1" H 4700 3875 40  0000 C CNN
 F 1 "DIODE" H 4700 3675 40  0000 C CNN
-F 2 "~" H 4700 3775 60  0000 C CNN
+F 2 "Diodes_SMD:D_0603" H 4700 3775 60  0001 C CNN
 F 3 "http://www.onsemi.com/pub_link/Collateral/MRA4003T3-D.PDF" H 4700 3775 60  0001 C CNN
 F 4 "1A, 1000V, SILICON, SIGNAL DIODE, ROHS COMPLIANT, COMPACT, PLASTIC, CASE 403D-02, SMA, 2 PIN" H 4700 3775 60  0001 C CNN "Characteristics"
@@
 F 0 "C1" H 5325 4275 40  0000 L CNN
 F 1 "47uF" H 5325 4075 40  0000 L CNN
-F 2 "~" H 5375 4025 30  0000 C CNN
+F 2 "ATMEGA328P-AU:QFP80P900X900X120-32N" H 5375 4025 30  0000 C CNN
 F 3 "http://images.ihscontent.net/vipimages/VipMasterIC/IC/BEYS/BEYSS04513/BEYSS04513-1.pdf" H 5275 4175 300 0001 C CNN
 F 4 "CAPACITOR, ALUMINUM ELECTROLYTIC, NON SOLID, POLARIZED, 50 V, 47 uF, SURFACE MOUNT, 3131, CHIP, ROHS COMPLIANT" H 5275 4175 60  0001 C CNN "Characteristics"
@@
 F 0 "C3" H 7075 4275 40  0000 L CNN
 F 1 "0.1 uF" H 7075 4075 40  0000 L CNN
-F 2 "~" H 7063 4025 30  0000 C CNN
+F 2 "" H 7063 4025 30  0001 C CNN
 F 3 "http://images.ihscontent.net/vipimages/VipMasterIC/IC/KEME/KEMES10043/KEMES10043-1.pdf" H 7025 4175 60  0001 C CNN
 F 4 "CAPACITOR, CERAMIC, MULTILAYER, 100 V, X7R, 0.1 uF, SURFACE MOUNT, 0805, CHIP, ROHS COMPLIANT" H 7025 4175 60  0001 C CNN "Characteristics"
@@
 F 0 "CON1" H 3725 4025 60  0000 C CNN
 F 1 "BARREL_JACK" H 3725 3575 60  0000 C CNN
-F 2 "~" H 3725 3775 60  0000 C CNN
+F 2 "" H 3725 3775 60  0001 C CNN
 F 3 "http://katalog.we-online.de/em/datasheet/6941xx106102.pdf" H 3725 3775 60  0001 C CNN
 F 4 "CONN PWR JACK DC RA SMD	" H 3725 3775 60  0001 C CNN "Characteristics"
@@
 F 0 "C2" H 6675 4275 40  0000 L CNN
 F 1 "47uF" H 6675 4075 40  0000 L CNN
-F 2 "~" H 6725 4025 30  0000 C CNN
+F 2 "" H 6725 4025 30  0001 C CNN
 F 3 "http://images.ihscontent.net/vipimages/VipMasterIC/IC/BEYS/BEYSS04513/BEYSS04513-1.pdf" H 6625 4175 300 0001 C CNN
 F 4 "CAPACITOR, ALUMINUM ELECTROLYTIC, NON SOLID, POLARIZED, 50 V, 47 uF, SURFACE MOUNT, 3131, CHIP, ROHS COMPLIANT" H 6625 4175 60  0001 C CNN "Characteristics"
@@
 F 0 "R1" V 7880 3625 40  0000 C CNN
 F 1 "510" V 7807 3626 40  0000 C CNN
-F 2 "~" V 7730 3625 30  0000 C CNN
+F 2 "" V 7730 3625 30  0001 C CNN
 F 3 "http://www.yageo.com/pdf/Pu-RC0805_51_PbFree_L_2.pdf" H 7800 3625 30  0001 C CNN
 F 4 "RESISTOR, METAL GLAZE/THICK FILM, 0.125W, 1%, 100ppm, 510ohm, SURFACE MOUNT, 0805" H 7800 3625 60  0001 C CNN "Characteristics"
@@
 F 0 "D2" H 7800 4225 50  0000 C CNN
 F 1 "LED" H 7800 4025 50  0000 C CNN
-F 2 "~" H 7800 4125 60  0000 C CNN
+F 2 "" H 7800 4125 60  0001 C CNN
 F 3 "http://www.osram-os.com/Graphics/XPic9/00078860_0.pdf" H 7800 4125 60  0001 C CNN
 F 4 "LED CHIPLED 570NM GREEN" H 7800 4125 60  0001 C CNN "Characteristics"
@@
 F 0 "U1" H 6125 3575 60  0000 C CNN
 F 1 "LD1117S50TR" H 5925 4075 60  0000 C CNN
-F 2 "" H 5925 3825 60  0000 C CNN
+F 2 "LD1117S50TR:SOT230P700X190-4N" H 5925 3825 60  0001 C CNN
 F 3 "http://www.st.com/st-web-ui/static/active/en/resource/technical/document/datasheet/CD00000544.pdf" H 5925 3825 60  0001 C CNN
 F 4 "5 V FIXED POSITIVE LDO REGULATOR, 1.2 V DROPOUT, PDSO3, ROHS COMPLIANT, SOT-223, 4 PIN" H 5925 3825 60  0001 C CNN "Characteristics"
