File: ArduinoProject/elektronics/sensorModulo_x4/sensorModulo.sch (KiCad schematic (older format))
At the start: 13 parts, among them J1 Conn_01x06_Female, U1 TCRT5000, U2 TCRT5000, U3 TCRT5000, U4 TCRT5000

Commit message: modulo vier
Parts:
- U1, U2, U3, U4: footprint (none) -> lib:TRTC5000
Changed lines of the file:
@@
 F 0 "U2" H 3850 4400 60  0000 C CNN
 F 1 "TCRT5000" H 3850 4550 60  0000 C CNN
-F 2 "" H 3850 4400 60  0001 C CNN
+F 2 "lib:TRTC5000" H 3850 4400 60  0001 C CNN
 F 3 "" H 3850 4400 60  0001 C CNN
 	1    3850 4400
@@
 F 0 "U1" H 3850 2800 60  0000 C CNN
 F 1 "TCRT5000" H 3850 2950 60  0000 C CNN
-F 2 "" H 3850 2800 60  0001 C CNN
+F 2 "lib:TRTC5000" H 3850 2800 60  0001 C CNN
 F 3 "" H 3850 2800 60  0001 C CNN
 	1    3850 2800
@@
 F 0 "U3" H 3925 5800 60  0000 C CNN
 F 1 "TCRT5000" H 3925 5950 60  0000 C CNN
-F 2 "" H 3925 5800 60  0001 C CNN
+F 2 "lib:TRTC5000" H 3925 5800 60  0001 C CNN
 F 3 "" H 3925 5800 60  0001 C CNN
 	1    3925 5800
@@
 F 0 "U4" H 3825 7025 60  0000 C CNN
 F 1 "TCRT5000" H 3825 7175 60  0000 C CNN
-F 2 "" H 3825 7025 60  0001 C CNN
+F 2 "lib:TRTC5000" H 3825 7025 60  0001 C CNN
 F 3 "" H 3825 7025 60  0001 C CNN
 	1    3825 7025
