File: ArduinoProject/elektronics/sensorModulo_x4/sensorModulo.sch (KiCad schematic (older format))
At the start: 13 parts, among them J1 Conn_01x06_Female, U1 TCRT5000, U2 TCRT5000, U3 TCRT5000, U4 TCRT5000

Commit message: modulo4x
Parts:
- J1: footprint Socket_Strips:Socket_Strip_Straight_1x06_Pitch2.00mm -> Socket_Strips:Socket_Strip_Straight_1x06_Pitch2.54mm
Changed lines of the file:
@@
 F 0 "J1" H 1550 5575 50  0000 C CNN
 F 1 "Conn_01x06_Female" H 1550 4875 50  0000 C CNN
-F 2 "Socket_Strips:Socket_Strip_Straight_1x06_Pitch2.00mm" H 1550 5275 50  0001 C CNN
+F 2 "Socket_Strips:Socket_Strip_Straight_1x06_Pitch2.54mm" H 1550 5275 50  0001 C CNN
 F 3 "" H 1550 5275 50  0001 C CNN
 	1    1550 5275

Commit message: sensorx4module
Parts:
- U1, U2, U3, U4: footprint (none) -> lib:TRTC5000
Changed lines of the file:
@@
 F 0 "U2" H 3850 4400 60  0000 C CNN
 F 1 "TCRT5000" H 3850 4550 60  0000 C CNN
-F 2 "" H 3850 4400 60  0001 C CNN
+F 2 "lib:TRTC5000" H 3850 4400 60  0001 C CNN
 F 3 "" H 3850 4400 60  0001 C CNN
 	1    3850 4400
@@
 F 0 "U1" H 3850 2800 60  0000 C CNN
 F 1 "TCRT5000" H 3850 2950 60  0000 C CNN
-F 2 "" H 3850 2800 60  0001 C CNN
+F 2 "lib:TRTC5000" H 3850 2800 60  0001 C CNN
 F 3 "" H 3850 2800 60  0001 C CNN
 	1    3850 2800
@@
 F 0 "U3" H 3925 5800 60  0000 C CNN
 F 1 "TCRT5000" H 3925 5950 60  0000 C CNN
-F 2 "" H 3925 5800 60  0001 C CNN
+F 2 "lib:TRTC5000" H 3925 5800 60  0001 C CNN
 F 3 "" H 3925 5800 60  0001 C CNN
 	1    3925 5800
@@
 F 0 "U4" H 3825 7025 60  0000 C CNN
 F 1 "TCRT5000" H 3825 7175 60  0000 C CNN
-F 2 "" H 3825 7025 60  0001 C CNN
+F 2 "lib:TRTC5000" H 3825 7025 60  0001 C CNN
 F 3 "" H 3825 7025 60  0001 C CNN
 	1    3825 7025
