File: ArduinoProject/elektronics/arduino_unoModulo_tot_32pin/Motor_Outputs.sch (KiCad schematic (older format))
At the start: 9 parts, among them X1 DG3XX-04-3.5

Commit message: arduino altered
Parts:
- D501, D502, D503, D504, D505, D506, D507, D508: footprint Diodes_SMD:D_0805 -> SK25AHM2G:DIOM5437X240N
Changed lines of the file:
@@
 F 0 "D501" H 4200 2900 50  0000 C CNN
 F 1 "D" H 4200 2700 50  0000 C CNN
-F 2 "Diodes_SMD:D_0805" H 4200 2800 50  0001 C CNN
+F 2 "SK25AHM2G:DIOM5437X240N" H 4200 2800 50  0001 C CNN
 F 3 "" H 4200 2800 50  0001 C CNN
 	1    4200 2800
@@
 F 0 "D503" H 4700 2900 50  0000 C CNN
 F 1 "D" H 4700 2700 50  0000 C CNN
-F 2 "Diodes_SMD:D_0805" H 4700 2800 50  0001 C CNN
+F 2 "SK25AHM2G:DIOM5437X240N" H 4700 2800 50  0001 C CNN
 F 3 "" H 4700 2800 50  0001 C CNN
 	1    4700 2800
@@
 F 0 "D505" H 5250 2900 50  0000 C CNN
 F 1 "D" H 5250 2700 50  0000 C CNN
-F 2 "Diodes_SMD:D_0805" H 5250 2800 50  0001 C CNN
+F 2 "SK25AHM2G:DIOM5437X240N" H 5250 2800 50  0001 C CNN
 F 3 "" H 5250 2800 50  0001 C CNN
 	1    5250 2800
@@
 F 0 "D507" H 5800 2900 50  0000 C CNN
 F 1 "D" H 5800 2700 50  0000 C CNN
-F 2 "Diodes_SMD:D_0805" H 5800 2800 50  0001 C CNN
+F 2 "SK25AHM2G:DIOM5437X240N" H 5800 2800 50  0001 C CNN
 F 3 "" H 5800 2800 50  0001 C CNN
 	1    5800 2800
@@
 F 0 "D502" H 4200 4400 50  0000 C CNN
 F 1 "D" H 4200 4200 50  0000 C CNN
-F 2 "Diodes_SMD:D_0805" H 4200 4300 50  0001 C CNN
+F 2 "SK25AHM2G:DIOM5437X240N" H 4200 4300 50  0001 C CNN
 F 3 "" H 4200 4300 50  0001 C CNN
 	1    4200 4300
@@
 F 0 "D504" H 4700 4400 50  0000 C CNN
 F 1 "D" H 4700 4200 50  0000 C CNN
-F 2 "Diodes_SMD:D_0805" H 4700 4300 50  0001 C CNN
+F 2 "SK25AHM2G:DIOM5437X240N" H 4700 4300 50  0001 C CNN
 F 3 "" H 4700 4300 50  0001 C CNN
 	1    4700 4300
@@
 F 0 "D506" H 5250 4400 50  0000 C CNN
 F 1 "D" H 5250 4200 50  0000 C CNN
-F 2 "Diodes_SMD:D_0805" H 5250 4300 50  0001 C CNN
+F 2 "SK25AHM2G:DIOM5437X240N" H 5250 4300 50  0001 C CNN
 F 3 "" H 5250 4300 50  0001 C CNN
 	1    5250 4300
@@
 F 0 "D508" H 5800 4400 50  0000 C CNN
 F 1 "D" H 5800 4200 50  0000 C CNN
-F 2 "Diodes_SMD:D_0805" H 5800 4300 50  0001 C CNN
+F 2 "SK25AHM2G:DIOM5437X240N" H 5800 4300 50  0001 C CNN
 F 3 "" H 5800 4300 50  0001 C CNN
 	1    5800 4300
