File: ArduinoProject/elektronics/arduino_unoModulo_tot_32pin/L298_Driver.sch (KiCad schematic (older format))
At the start: 6 parts, among them U301 74AHC1G04, U302 L298D, U303 74AHC1G04

Commit message: diode changed
Parts:
- C301: footprint Capacitors_SMD:CP_Elec_5x5.3 -> Capacitors_SMD:CP_Elec_4x5.3
Changed lines of the file:
@@
 F 0 "C301" H 4175 3750 50  0000 L CNN
 F 1 "100uF.25V" H 3750 3550 50  0000 L CNN
-F 2 "Capacitors_SMD:CP_Elec_5x5.3" H 4150 3650 50  0001 C CNN
+F 2 "Capacitors_SMD:CP_Elec_4x5.3" H 4150 3650 50  0001 C CNN
 F 3 "" H 4150 3650 50  0001 C CNN
 	1    4150 3650

Commit message: vias dik
Parts:
- removed C301: 100uF.25V, Capacitors_SMD:CP_Elec_4x5.3, symbol CP1
- added CP301: 100uF.25V, Capacitors_SMD:CP_Elec_4x5.3, symbol CP
Connections:
- net GND: now also CP301.2
- net PWRIN: now also CP301.1
Changed lines of the file:
@@
-$EndComp
-$Comp
-L CP1 C301
-U 1 1 5A964B4A
-P 4150 3650
-F 0 "C301" H 4175 3750 50  0000 L CNN
-F 1 "100uF.25V" H 3750 3550 50  0000 L CNN
-F 2 "Capacitors_SMD:CP_Elec_4x5.3" H 4150 3650 50  0001 C CNN
-F 3 "" H 4150 3650 50  0001 C CNN
-	1    4150 3650
-	1    0    0    -1
 $EndComp
 $Comp
@@
 	1    0    0    -1
 $EndComp
+$Comp
+L CP CP301
+U 1 1 5AABE897
+P 4150 3650
+F 0 "CP301" H 4175 3750 50  0000 L CNN
+F 1 "100uF.25V" H 4175 3550 50  0000 L CNN
+F 2 "Capacitors_SMD:CP_Elec_4x5.3" H 4188 3500 50  0001 C CNN
+F 3 "" H 4150 3650 50  0001 C CNN
+	1    4150 3650
+	1    0    0    -1
+$EndComp
