File: ArduinoProject/elektronics/arduino_unoModulo_tot_32pin/L298_Driver.sch (KiCad schematic (older format))
At the start: 6 parts, among them U301 74AHC1G04, U302 L298D, U303 74AHC1G04

Commit message: changes made
Parts:
- CP301: footprint Capacitors_SMD:CP_Elec_4x5.3 -> Capacitors_SMD:CP_Elec_6.3x5.3
Connections:
- net +5V: now also U303.5 (VCC); no longer U303.3 (GND)
- net GND: now also U303.3 (GND); no longer U303.5 (VCC)
Other:
- moved on the sheet: C303
Changed lines of the file:
@@
 L GND #PWR07
 U 1 1 5A8D7873
-P 7800 3250
-F 0 "#PWR07" H 7800 3000 50  0001 C CNN
-F 1 "GND" H 7800 3100 50  0000 C CNN
-F 2 "" H 7800 3250 50  0001 C CNN
-F 3 "" H 7800 3250 50  0001 C CNN
-	1    7800 3250
-	1    0    0    -1
+P 7800 2700
+F 0 "#PWR07" H 7800 2450 50  0001 C CNN
+F 1 "GND" H 7800 2550 50  0000 C CNN
+F 2 "" H 7800 2700 50  0001 C CNN
+F 3 "" H 7800 2700 50  0001 C CNN
+	1    7800 2700
+	-1   0    0    1
 $EndComp
 $Comp
@@
 L C C303
 U 1 1 5A9642A9
-P 8100 2600
-F 0 "C303" H 8125 2700 50  0000 L CNN
-F 1 "0.1uF" H 8125 2500 50  0000 L CNN
-F 2 "Capacitors_SMD:C_0805" H 8138 2450 50  0001 C CNN
-F 3 "" H 8100 2600 50  0001 C CNN
-	1    8100 2600
+P 8350 3500
+F 0 "C303" H 8375 3600 50  0000 L CNN
+F 1 "0.1uF" H 8375 3400 50  0000 L CNN
+F 2 "Capacitors_SMD:C_0805" H 8388 3350 50  0001 C CNN
+F 3 "" H 8350 3500 50  0001 C CNN
+	1    8350 3500
 	0    1    1    0
 $EndComp
@@
 L GND #PWR09
 U 1 1 5A964733
-P 8400 2600
-F 0 "#PWR09" H 8400 2350 50  0001 C CNN
-F 1 "GND" H 8400 2450 50  0000 C CNN
-F 2 "" H 8400 2600 50  0001 C CNN
-F 3 "" H 8400 2600 50  0001 C CNN
-	1    8400 2600
+P 8650 3500
+F 0 "#PWR09" H 8650 3250 50  0001 C CNN
+F 1 "GND" H 8650 3350 50  0000 C CNN
+F 2 "" H 8650 3500 50  0001 C CNN
+F 3 "" H 8650 3500 50  0001 C CNN
+	1    8650 3500
 	0    -1   -1   0
 $EndComp
@@
 L +5V #PWR013
 U 1 1 5A9E6DF9
-P 7800 2450
-F 0 "#PWR013" H 7800 2300 50  0001 C CNN
-F 1 "+5V" H 7800 2590 50  0000 C CNN
-F 2 "" H 7800 2450 50  0001 C CNN
-F 3 "" H 7800 2450 50  0001 C CNN
-	1    7800 2450
+P 8050 3350
+F 0 "#PWR013" H 8050 3200 50  0001 C CNN
+F 1 "+5V" H 8050 3490 50  0000 C CNN
+F 2 "" H 8050 3350 50  0001 C CNN
+F 3 "" H 8050 3350 50  0001 C CNN
+	1    8050 3350
 	1    0    0    -1
 $EndComp
@@
 	3350 3550 3350 3500
 Wire Wire Line
-	7800 3250 7800 3200
-Wire Wire Line
 	3350 2425 3350 3100
-Wire Wire Line
-	7800 2450 7800 2800
 Connection ~ 3350 2600
 Wire Wire Line
@@
 	6750 3300 6750 2200
 Wire Wire Line
-	7950 2600 7800 2600
-Connection ~ 7800 2600
-Wire Wire Line
-	8400 2600 8250 2600
+	7800 3500 8200 3500
+Connection ~ 8050 3500
+Wire Wire Line
+	8650 3500 8500 3500
 Wire Wire Line
 	8200 3000 8450 3000
@@
 F 0 "CP301" H 4175 3750 50  0000 L CNN
 F 1 "100uF.25V" H 4175 3550 50  0000 L CNN
-F 2 "Capacitors_SMD:CP_Elec_4x5.3" H 4188 3500 50  0001 C CNN
+F 2 "Capacitors_SMD:CP_Elec_6.3x5.3" H 4188 3500 50  0001 C CNN
 F 3 "" H 4150 3650 50  0001 C CNN
 	1    4150 3650
 	1    0    0    -1
 $EndComp
+Wire Wire Line
+	7800 2800 7800 2700
+Wire Wire Line
+	7800 3500 7800 3200
+Wire Wire Line
+	8050 3350 8050 3500
 $EndSCHEMATC
