File: ArduinoProject/elektronics/arduino_unoModulo_tot_32pin/Arduino_Uno_R3_From_Scratch.kicad_pcb (KiCad board)
At the start: 2 copper layers, 68.9 x 47.8 mm, 36 parts, among them IC401 MC33269ST-5.OT3, IC402 MC33269ST-5.OT3, J201 POWER, J202 IOL, J203 IOL, J204 IOL, SW601 RESET_SWITCH, U301 74AHC1G04, U302 L298D, U303 74AHC1G04, U601 ATMEGA328P-MU20, X1 DG3XX-04-3.5, X2 DG3XX-02-3.5, Y601 Crystal

Commit message: vias dik
Parts:
- moved C302 0.24 mm to (151.8, 137.2)
Routing:
- net +5V: track 241.0 -> 243.7 mm
- net /ATMEGA328P/PWMA: track 47.5 -> 49.9 mm
- net /L298_Driver./PWRIN: track 83.5 -> 84.4 mm

Commit message: changes made
Parts:
- removed C301: 100uF.25V, Capacitors_SMD:CP_Elec_5x5.3
- added CP301: 100uF.25V, Capacitors_SMD:CP_Elec_6.3x5.3, F.Cu at (151.2, 127.5)
- D401: footprint Diodes_SMD:D_MicroMELF_Hadsoldering -> Diodes_SMD:D_MiniMELF_Handsoldering
- PC401, PC402: footprint Capacitors_SMD:CP_Elec_4x5.3 -> Capacitors_SMD:CP_Elec_6.3x5.3
- moved C602 6.27 mm to (190.7, 104.8), turned to 270 degrees
- moved X2 2.64 mm to (154.0, 97.7)
- moved D401 1.99 mm to (162.5, 98.7), turned to 180 degrees
- moved U303 1.98 mm to (176.4, 133.4), turned to 180 degrees
- moved PC402 1.85 mm to (181.6, 106.9), turned to 0 degrees
- moved PC401 0.38 mm to (172.6, 105.9), turned to 90 degrees
- turned C401 to 180 degrees
Connections:
- C401 pad 1: +5V -> GND
- C401 pad 2: GND -> +5V
- U303 pad 3: +5V -> GND
- U303 pad 5: GND -> +5V
Routing:
- net Net-(U302-Pad15): track 23.7 -> 8.11 mm
- net /L298_Driver./PWRIN: track 84.4 -> 73.6 mm, vias 0 -> 1
- net /Headers/VIN: track 35.2 -> 30.8 mm
- net GND: track 404.7 -> 408.8 mm
- net 328P_ICSP_SCK: track 155.5 -> 159.4 mm
- net +5V: track 243.7 -> 246.8 mm
Other:
- net class fortymill: clearance 0.2 -> 0.1

Commit message: chaged printplaat'
Parts:
- moved C603 9.78 mm to (189.8, 127.7), turned to 180 degrees
Routing:
- net GND: track 408.8 -> 380.8 mm, vias 4 -> 5
- net Net-(C603-Pad2): track 36.8 -> 14.5 mm, vias 0 -> 2
- net 328P_ICSP_SCK: track 159.4 -> 158.2 mm
- net /ATMEGA328P/AD6: track 52.3 -> 51.4 mm
- added copper zone on F.Cu, net GND
Other:
- outline, holes or cut-outs redrawn
