File: ArduinoProject/elektronics/arduino_unoModulo_second_version/Arduino_Uno_R3_From_Scratch.kicad_pcb (KiCad board)
At the start: 2 copper layers, 62 x 47.8 mm, 35 parts, among them IC401 MC33269ST-5.OT3, IC402 MC33269ST-5.OT3, J201 digitaal/voltages, J202 digital/gnd/aref, J203 analog, SW601 RESET_SWITCH, U301 74AHC1G04, U302 L298D, U303 74AHC1G04, U601 ATMEGA328P-MU20, X1 DG3XX-04-3.5, X2 DG3XX-02-3.5, Y601 Crystal

Commit message: second printplaat version added2
Connections:
- U601 pad 10: /ATMEGA328P/DIRB -> /ATMEGA328P/PWMA
- U601 pad 11: /ATMEGA328P/PWMA -> /ATMEGA328P/DIRB
Routing:
- net GND: track 72.6 -> 78.8 mm
- net +5V: track 165.8 -> 169.0 mm
- net /ATMEGA328P/DIRB: track 18.1 -> 20.8 mm
- net /ATMEGA328P/PWMA: track 39.2 -> 39.9 mm, vias 0 -> 2
- net /L298_Driver./OUT3: track 59.3 -> 58.6 mm
- net /L298_Driver./OUT1: track 61.3 -> 60.8 mm
Other:
- outline, holes or cut-outs redrawn
